File: hardware/mainboard/power.kicad_sch (KiCad schematic)
At the start: 21 parts, among them J1 Eurorack Power, U1 LD1117-3.3, U2 LM4040DBZ-10

Commit message: exclude components from BOM
excluded:
- J11 (alternate USB connection)
- test points
Parts:
- TP1, TP2, TP3: now left out of the parts list
Changed lines of the file:
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@@
 		(unit 1)
 		(exclude_from_sim no)
-		(in_bom yes)
+		(in_bom no)
 		(on_board yes)
 		(dnp no)
@@
 		(unit 1)
 		(exclude_from_sim no)
-		(in_bom yes)
+		(in_bom no)
 		(on_board yes)
 		(dnp no)
@@
 		(unit 1)
 		(exclude_from_sim no)
-		(in_bom yes)
-		(on_board yes)
-		(dnp no)
+		(in_bom no)
+		(on_board yes)
+		(dnp no)
