File: hardware/mainboard/outputmixer.kicad_sch (KiCad schematic)
At the start: 15 parts, among them J10 MIX, J9 EXT, U12 TL074, U8 TL074

Commit message: add alternate for TL074
added TL074CPWR as alternate in addition to TL074CPW
Parts:
- U8: MPN TL074CPW -> TL074CPW, TL074CPWR
Changed lines of the file:
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@@
 			)
 		)
-		(property "MPN" "TL074CPW"
+		(property "MPN" "TL074CPW, TL074CPWR"
 			(at 140.97 87.63 0)
 			(effects
